Commit message: first commit

File: install/xarm_1s_description/share/xarm_1s_description/urdf/xarm_1s.urdf.xacro (robot description, xacro)
@@ -233,52 +233,5 @@
   </joint>
   <link name="depth" />
-  <!-- TO-DO: move out to separate file -->
-  <ros2_control name="xarm_1s" type="system">
-    <hardware>
-      <!--plugin>ros2_control_xarm_1s/XArm1SSystemHardware</plugin-->
-      <plugin>mock_components/GenericSystem</plugin>
-    </hardware>
-    <joint name="arm6">
-      <command_interface name="position">
-        <param name="min">-2.09439435</param>
-        <param name="max">2.09439435</param>
-      </command_interface>
-      <state_interface name="position"/>
-    </joint>
-    <joint name="arm5">
-      <command_interface name="position">
-        <param name="min">-2.09439435</param>
-        <param name="max">2.09439435</param>
-      </command_interface>
-      <state_interface name="position"/>
-    </joint>
-    <joint name="arm4">
-      <command_interface name="position">
-        <param name="min">-2.09439435</param>
-        <param name="max">2.09439435</param>
-      </command_interface>
-      <state_interface name="position"/>
-    </joint>
-    <joint name="arm3">
-      <command_interface name="position">
-        <param name="min">-2.09439435</param>
-        <param name="max">2.09439435</param>
-      </command_interface>
-      <state_interface name="position"/>
-    </joint>
-    <joint name="arm2">
-      <command_interface name="position">
-        <param name="min">-2.09439435</param>
-        <param name="max">2.09439435</param>
-      </command_interface>
-      <state_interface name="position"/>
-    </joint>
-    <joint name="arm1">
-      <command_interface name="position">
-        <param name="min">0</param>
-        <param name="max">0.8464847</param>
-      </command_interface>
-      <state_interface name="position"/>
-    </joint>
-  </ros2_control>
+  <xacro:include filename="$(find xarm_1s_description)/urdf/control/xarm_1s.ros2_control.xacro" />
+  <xacro:xarm_1s_ros2_control name="xarm_1s"/>
 </robot>
