Commit message: bringup

File: install/xarm_1s_description/share/xarm_1s_description/urdf/control/xarm_1s.ros2_control.xacro (robot description, xacro)
@@ -1,77 +1 @@
-<?xml version="1.0"?>
-<robot xmlns:xacro="http://www.ros.org/wiki/xacro">
-    <!-- use_mock:=true  → 시뮬레이션 (RViz만)  -->
-    <!-- use_mock:=false → 실제 로봇 (HID 통신) -->
-    <xacro:arg name="use_mock" default="true"/>
-    <xacro:macro name="xarm_1s_ros2_control" params="name">
-        <ros2_control name="${name}" type="system">
-            <hardware>
-                <xacro:if value="$(arg use_mock)">
-                    <plugin>mock_components/GenericSystem</plugin>
-                </xacro:if>
-                <xacro:unless value="$(arg use_mock)">
-                    <plugin>xarm_1s_hardware/XArm1SHardwareInterface</plugin>
-                    <!-- Hiwonder xArm VID/PID -->
-                    <param name="vid">0x0483</param>
-                    <param name="pid">0x5750</param>
-                </xacro:unless>
-            </hardware>
-            <joint name="arm6">
-                <command_interface name="position">
-                    <param name="min">-2.09439435</param>
-                    <param name="max">2.09439435</param>
-                </command_interface>
-                <state_interface name="position"/>
-            </joint>
-            <joint name="arm5">
-                <command_interface name="position">
-                    <param name="min">-2.09439435</param>
-                    <param name="max">2.09439435</param>
-                </command_interface>
-                <state_interface name="position"/>
-            </joint>
-            <joint name="arm4">
-                <command_interface name="position">
-                    <param name="min">-2.09439435</param>
-                    <param name="max">2.09439435</param>
-                </command_interface>
-                <state_interface name="position"/>
-            </joint>
-            <joint name="arm3">
-                <command_interface name="position">
-                    <param name="min">-2.09439435</param>
-                    <param name="max">2.09439435</param>
-                </command_interface>
-                <state_interface name="position"/>
-            </joint>
-            <joint name="arm2">
-                <command_interface name="position">
-                    <param name="min">-2.09439435</param>
-                    <param name="max">2.09439435</param>
-                </command_interface>
-                <state_interface name="position"/>
-            </joint>
-            <joint name="arm1">
-                <command_interface name="position">
-                    <param name="min">0</param>
-                    <param name="max">0.8464847</param>
-                </command_interface>
-                <state_interface name="position"/>
-                <!--속도 추가 그리퍼 컨트롤러 에러 원인??-->
-                <state_interface name="velocity"/>
-            </joint>
-            <joint name="arm1_left">
-                <mimic joint="arm1" multiplier="-1" offset="0"/>
-                <state_interface name="position"/>
-            </joint>
-            <joint name="arm0">
-                <mimic joint="arm1" multiplier="-1.01" offset="-0.3"/>
-                <state_interface name="position"/>
-            </joint>
-            <joint name="arm0_left">
-                <mimic joint="arm1" multiplier="1.01" offset="0.3"/>
-                <state_interface name="position"/>
-            </joint>
-        </ros2_control>
-    </xacro:macro>
-</robot>
+/home/hyeon/xarm_ws/src/xarm_1s_description/urdf/control/xarm_1s.ros2_control.xacro

File: install/xarm_1s_description/share/xarm_1s_description/urdf/xarm_1s.urdf.xacro (robot description, xacro)
@@ -1,237 +1 @@
-<?xml version="1.0" ?>
-<robot xmlns:xacro="http://www.ros.org/wiki/xacro" name="xarm_1s">
-  <material name="black">
-    <color rgba="0.2 0.2 0.2 1"/>
-  </material>
-  <material name="blue">
-    <color rgba="0.3 0.5 0.9 1.0"/>
-  </material>
-  <link name="world"/>
-  <joint name="world_joint" type="fixed">
-    <parent link="world"/>
-    <child link="base_link"/>
-    <origin rpy="0.0 0.0 0.0" xyz="0.0 0.0 0.0"/>
-  </joint>
-  <link name="base_link">
-    <visual>
-      <origin rpy="0 0 0" xyz="0.0 0.0 0.0" />
-      <geometry>
-        <mesh filename="package://xarm_1s_description/meshes/base.stl" scale="1.0 1.0 1.0" />
-      </geometry>
-      <material name="blue" />
-    </visual>
-    <collision>
-      <origin rpy="0 0 0" xyz="0 0 0" />
-      <geometry>
-        <mesh filename="package://xarm_1s_description/meshes/base_collision.stl" scale="1.0 1.0 1.0" />
-      </geometry>
-    </collision>
-  </link>
-  <joint name="arm6" type="revolute">
-    <limit effort="1000" lower="-2.1" upper="2.1" velocity="1.0" />
-    <parent link="base_link"/>
-    <child link="link6"/>
-    <origin rpy="0.0 0.0 0.0" xyz="0.0 0.0 0.043"/>
-    <axis xyz="0 0 1"/>
-  </joint>
-  <link name="link6">
-    <visual>
-      <origin rpy="0 0 0" xyz="0.0 0.0 0.0" />
-      <geometry>
-        <mesh filename="package://xarm_1s_description/meshes/link6.stl" scale="1.0 1.0 1.0" />
-      </geometry>
-      <material name="blue" />
-    </visual>
-    <collision>
-      <origin rpy="0 0 0" xyz="0 0 0" />
-      <geometry>
-        <mesh filename="package://xarm_1s_description/meshes/link6_collision.stl" scale="1.0 1.0 1.0" />
-      </geometry>
-    </collision>
-  </link>
-  <joint name="arm5" type="revolute">
-    <limit effort="1000" lower="-1.5708" upper="1.5708" velocity="1.0" />
-    <parent link="link6"/>
-    <child link="link5"/>
-    <origin rpy="0.0 0.0 0.0" xyz="0.002 0.0 0.032"/>
-    <axis xyz="0 1 0"/>
-  </joint>
-  <link name="link5">
-    <visual>
-      <origin rpy="0 0 0" xyz="0.0 0.0 0.0" />
-      <geometry>
-        <mesh filename="package://xarm_1s_description/meshes/link5.stl" scale="1.0 1.0 1.0" />
-      </geometry>
-      <material name="blue" />
-    </visual>
-    <collision>
-      <origin rpy="0 0 0" xyz="0 0 0" />
-      <geometry>
-        <mesh filename="package://xarm_1s_description/meshes/link5_collision.stl" scale="1.0 1.0 1.0" />
-      </geometry>
-    </collision>
-  </link>
-  <joint name="arm4" type="revolute">
-    <limit effort="1000" lower="-2.09" upper="2.09" velocity="1.0" />
-    <parent link="link5"/>
-    <child link="link4"/>
-    <origin rpy="0.0 0.0 0.0" xyz="0.0 0.0 0.09775"/>
-    <axis xyz="0 1 0"/>
-  </joint>
-  <link name="link4">
-    <visual>
-      <origin rpy="0 0 0" xyz="0.0 0.0 0.0" />
-      <geometry>
-        <mesh filename="package://xarm_1s_description/meshes/link4.stl" scale="1.0 1.0 1.0" />
-      </geometry>
-      <material name="black" />
-    </visual>
-    <collision>
-      <origin rpy="0 0 0" xyz="0 0 0" />
-      <geometry>
-        <mesh filename="package://xarm_1s_description/meshes/link4_collision.stl" scale="1.0 1.0 1.0" />
-      </geometry>
-    </collision>
-  </link>
-  <joint name="arm3" type="revolute">
-    <limit effort="1000" lower="-1.85" upper="2.07" velocity="1.0" />
-    <parent link="link4"/>
-    <child link="link3"/>
-    <origin rpy="0.0 0.0 0.0" xyz="0.0 0.0 0.099"/>
-    <axis xyz="0 1 0"/>
-  </joint>
-  <link name="link3">
-    <visual>
-      <origin rpy="0 0 0" xyz="0.0 0.0 0.0" />
-      <geometry>
-        <mesh filename="package://xarm_1s_description/meshes/link3.stl" scale="1.0 1.0 1.0" />
-      </geometry>
-      <material name="blue" />
-    </visual>
-    <collision>
-      <origin rpy="0 0 0" xyz="0 0 0" />
-      <geometry>
-        <mesh filename="package://xarm_1s_description/meshes/link3_collision.stl" scale="1.0 1.0 1.0" />
-      </geometry>
-    </collision>
-  </link>
-  <joint name="arm2" type="revolute">
-    <limit effort="1000" lower="-1.95" upper="1.95" velocity="1.0" />
-    <parent link="link3"/>
-    <child link="link2"/>
-    <origin rpy="0.0 0.0 0.0" xyz="-0.00125 0.0 0.050"/>
-    <axis xyz="0 0 1"/>
-  </joint>
-  <link name="link2">
-    <visual>
-      <origin rpy="0 0 0" xyz="0.0 0.0 0.0" />
-      <geometry>
-        <mesh filename="package://xarm_1s_description/meshes/link2.stl" scale="1.0 1.0 1.0" />
-      </geometry>
-      <material name="black" />
-    </visual>
-    <collision>
-      <origin rpy="0 0 0" xyz="0 0 0" />
-      <geometry>
-        <mesh filename="package://xarm_1s_description/meshes/link2_collision.stl" scale="1.0 1.0 1.0" />
-      </geometry>
-    </collision>
-  </link>
-  <joint name="arm1" type="revolute">
-    <limit effort="1000" lower="0" upper="1.8326" velocity="1.0" />
-    <parent link="link2"/>
-    <child link="link1"/>
-    <origin xyz="-0.0015 -0.014 0.0315" rpy="0.0 0.0 0.0" />
-    <axis xyz="1 0 0"/>
-  </joint>
-  <link name="link1">
-    <visual>
-      <origin rpy="0 0 0" xyz="0.0 0.0 0.0" />
-      <geometry>
-        <mesh filename="package://xarm_1s_description/meshes/link1.stl" scale="1.0 1.0 1.0" />
-      </geometry>
-      <material name="black" />
-    </visual>
-    <collision>
-      <origin rpy="0 0 0" xyz="0 0 0" />
-      <geometry>
-        <mesh filename="package://xarm_1s_description/meshes/link1_collision.stl" scale="1.0 1.0 1.0" />
-      </geometry>
-    </collision>
-  </link>
-  <joint name="arm1_left" type="continuous">
-    <parent link="link2"/>
-    <child link="link1_left"/>
-    <origin xyz="-0.0015 0.014 0.0315" rpy="0.0 0.0 0.0" />
-    <axis xyz="1 0 0"/>
-    <mimic joint="arm1" multiplier="-1" offset="0" />
-  </joint>
-  <link name="link1_left">
-    <visual>
-      <origin rpy="0 0 0" xyz="0.0 0.0 0.0" />
-      <geometry>
-        <mesh filename="package://xarm_1s_description/meshes/link1_left.stl" scale="1.0 1.0 1.0" />
-      </geometry>
-      <material name="black" />
-    </visual>
-    <collision>
-      <origin rpy="0 0 0" xyz="0 0 0" />
-      <geometry>
-        <mesh filename="package://xarm_1s_description/meshes/link1_left_collision.stl" scale="1.0 1.0 1.0" />
-      </geometry>
-    </collision>
-  </link>
-  <joint name="arm0" type="continuous">
-    <parent link="link1"/>
-    <child link="link0"/>
-    <origin xyz="-0.0023 0.0 0.0305" rpy="0.0 0.0 0.0" />
-    <axis xyz="1 0 0"/>
-    <mimic joint="arm1" multiplier="-1.01" offset="-0.3" />
-  </joint>
-  <link name="link0">
-    <visual>
-      <origin rpy="0 0 0" xyz="0.0 0.0 0.0" />
-      <geometry>
-        <mesh filename="package://xarm_1s_description/meshes/link0.stl" scale="1.0 1.0 1.0" />
-      </geometry>
-      <material name="black" />
-    </visual>
-    <collision>
-      <origin rpy="0 0 0" xyz="0 0 0" />
-      <geometry>
-        <mesh filename="package://xarm_1s_description/meshes/link0_collision.stl" scale="1.0 1.0 1.0" />
-      </geometry>
-    </collision>
-  </link>
-  <joint name="arm0_left" type="continuous">
-    <parent link="link1_left"/>
-    <child link="link0_left"/>
-    <origin xyz="-0.0023 0.0 0.0305" rpy="0.0 0.0 0.0" />
-    <axis xyz="1 0 0"/>
-    <mimic joint="arm1" multiplier="1.01" offset="0.3" />
-  </joint>
-  <link name="link0_left">
-    <visual>
-      <origin rpy="0 0 0" xyz="0.0 0.0 0.0" />
-      <geometry>
-        <mesh filename="package://xarm_1s_description/meshes/link0_left.stl" scale="1.0 1.0 1.0" />
-      </geometry>
-      <material name="black" />
-    </visual>
-    <collision>
-      <origin rpy="0 0 0" xyz="0 0 0" />
-      <geometry>
-        <mesh filename="package://xarm_1s_description/meshes/link0_left_collision.stl" scale="1.0 1.0 1.0" />
-      </geometry>
-    </collision>
-  </link>
-  <!-- TO-DO: move out to separate file -->
-  <joint name="depth_joint" type="fixed">
-    <parent link="link2"/>
-    <child link="depth"/>
-    <origin rpy="-1.5708 0 -1.5708" xyz="0.044 -0.0115 0.045"/>
-  </joint>
-  <link name="depth" />
-  <xacro:include filename="$(find xarm_1s_description)/urdf/control/xarm_1s.ros2_control.xacro" />
-  <xacro:xarm_1s_ros2_control name="xarm_1s"/>
-</robot>
+/home/hyeon/xarm_ws/src/xarm_1s_description/urdf/xarm_1s.urdf.xacro
